Commit message: exercise 5 added

File: resource/a1/urdf/a1.urdf (robot description, URDF)
Before this commit: robot a1_description, 19 links, 18 joints
Links:
- removed link FL_calf
- removed link FL_foot
- removed link FL_hip
- removed link FL_thigh
- removed link RL_calf
- removed link RL_foot
- removed link RL_hip
- removed link RL_thigh
- removed link RR_calf
- removed link RR_foot
- removed link RR_hip
- removed link RR_thigh
Joints:
- removed joint FL_calf_joint
- removed joint FL_foot_fixed
- removed joint FL_hip_joint
- removed joint FL_thigh_joint
- removed joint RL_calf_joint
- removed joint RL_foot_fixed
- removed joint RL_hip_joint
- removed joint RL_thigh_joint
- removed joint RR_calf_joint
- removed joint RR_foot_fixed
- removed joint RR_hip_joint
- removed joint RR_thigh_joint
